Commit message: Added GP225 Support Package for URDF
*Added a GP225 support package that was forked from Motoman's official github repo, will update with AIMS GP225 later.

File: forgescan_support/urdf/scene.urdf.xacro (robot description, xacro)
@@ -15,6 +15,6 @@
     <!-- Robot -->
     <xacro:include filename="$(find motoman_resources)/urdf/common_materials.xacro"/>
-    <xacro:include filename="$(find motoman_ms210_support)/urdf/ms210.xacro" />
-    <joint name="fix_origin_ms210" type="fixed">
+    <xacro:include filename="$(find motoman_gp225_support)/urdf/gp225.xacro" />
+    <joint name="fix_origin_gp225" type="fixed">
       <origin xyz="0 0 0.127" rpy="0 0 0"/>
       <parent link="world"/>
@@ -80,5 +80,5 @@
   <joint name="compliance_device_joint" type="fixed">
     <origin xyz="0 0 0" rpy="0 0 0"/>
-    <parent link="link_6_t"/>
+    <parent link="flange"/>
     <child link="compliance_device"/>
   </joint>
